Commit message: Added .rviz file, updated measurements in URDF file

File: urdf/virat.urdf (robot description, URDF)
Before this commit: robot origins, 4 links, 3 joints
Joints:
- joint castor_joint: axis 0 1 0 -> (none); origin xyz=0.48 0 0 -> xyz=0.48 0 0.02; type continuous -> fixed

Commit message: Added inertial and collision attributes to components

File: urdf/virat.urdf (robot description, URDF)
Before this commit: robot origins, 4 links, 3 joints
Links:
- removed link front_castor
- removed link left_wheel
- removed link right_wheel
- added link base_footprint
- added link front_castor_link, mass 0.2; collision mesh filename=package://virat_description/meshes/wheels/castors1.dae; visual mesh filename=package://virat_description/meshes/wheels/castors1.dae
- added link left_wheel_link, mass 1.0; collision mesh filename=package://virat_description/meshes/wheels/tyre1.dae; visual mesh filename=package://virat_description/meshes/wheels/tyre1.dae
- added link right_wheel_link, mass 1.0; collision mesh filename=package://virat_description/meshes/wheels/tyre1.dae; visual mesh filename=package://virat_description/meshes/wheels/tyre1.dae
- link base_link: mass None -> 6.0; geometry collision mesh filename=package://virat_description/meshes/body/bot2.dae; visual mesh filename=package://virat_description/meshes/body/bot2.dae
Joints:
- removed joint castor_joint
- removed joint left_axle
- removed joint right_axle
- added joint base_joint: type fixed, parent base_footprint, child base_link, origin xyz=0 0 0 rpy=0 0 0
- added joint front_castor_joint: type fixed, parent base_link, child front_castor_link, origin xyz=0.48 0 0.02
- added joint left_wheel_joint: type continuous, parent base_link, child left_wheel_link, origin xyz=0 0.323 0, axis 0 1 0
- added joint right_wheel_joint: type continuous, parent base_link, child right_wheel_link, origin xyz=0 -0.323 0, axis 0 1 0

Commit message: Added Gazebo differential drive plugin in virat.urdf

File: urdf/virat.urdf (robot description, URDF)
Before this commit: robot virat, 5 links, 4 joints
Links:
- link base_link: mass 6.0 -> 60.0
- link front_castor_link: mass 0.2 -> 2
- link left_wheel_link: mass 1.0 -> 10.0
- link right_wheel_link: mass 1.0 -> 10.0

Commit message: Updated values in URDF file

File: urdf/virat.urdf (robot description, URDF)
Before this commit: robot virat, 5 links, 4 joints
Links:
- link base_link: mass 60.0 -> 200
- link left_wheel_link: mass 10.0 -> 10
- link right_wheel_link: mass 10.0 -> 10

Commit message: Updated the physical values of robot (mass and inertias) to make the motion look more realistic
Currently, the values are not at all physically correct, but it at least works in simulation.
FIXME: Get better values, which are more closer to the real values, and also perform well in the simulation.

File: urdf/virat.urdf (robot description, URDF)
Before this commit: robot virat, 5 links, 4 joints
Links:
- link base_link: mass 200 -> 1.5
- link front_castor_link: mass 2 -> 1
- link left_wheel_link: mass 10 -> 0.4
- link right_wheel_link: mass 10 -> 0.4

Commit message: Added link and joint for top camera
TODO: Need to integrate this with Gazebo camera plugin

File: urdf/virat.urdf (robot description, URDF)
Before this commit: robot virat, 5 links, 4 joints
Links:
- added link camera_link; visual box size=0.05 0.05 0.05
Joints:
- added joint camera_joint: type fixed, parent base_link, child camera_link, origin xyz=0.72 0 1.18 rpy=0 0.45 0

Commit message: Added launch file for RVIZ, updated virat.rviz, included camera Gazebo plugin in virat.urdf
TODO: Try to remove a blue patch which appears when viewing raw camera output

File: urdf/virat.urdf (robot description, URDF)
Before this commit: robot virat, 6 links, 5 joints
Joints:
- joint camera_joint: origin xyz=0.72 0 1.18 rpy=0 0.45 0 -> xyz=0.73 0 1.18 rpy=0 0.45 0

Commit message: Changed node name to avoid collision, removed virat prefix used in frame

File: urdf/virat.urdf (robot description, URDF)
Before this commit: robot virat, 6 links, 5 joints
Links:
- removed link base_footprint
- added link dummy_link
Joints:
- joint base_joint: parent base_footprint -> dummy_link
